File: kicad/amp/amp_compact.kicad_pcb (KiCad board)
At the start: 2 copper layers, 100 x 85 mm, 112 parts, among them J1 DC 12V IN, J2 IN L-G-R, J3 SPK L, J4 SPK R, Q1001 BC547, Q1002 BC547, Q1003 BC557, Q1004 BD139, Q1005 BD140, Q1006 BC547, Q2001 BC547, Q2002 BC547, Q2003 BC557, Q2004 BD139, Q2005 BD140, Q2006 BC547

Commit message: Compact amp: title between the channels, revision at the bottom edge, URL on the back silkscreen; release copies the compact board
Other:
- board text added: "STEREO AMP 12V"
- board text added: "STEREO AMP 12V compact 100 x 85 mm CC BY-NC-SA 4.0"
- board text added: "github.com/lahirunirmalx/discrete-stereo-amp v1.1 2026-10"
- board text added: "v1.1 2026-10"
- board text removed: "STEREO AMP 12V v1.1 2026-10"
- board text removed: "github.com/lahirunirmalx/discrete-stereo-amp"
