File: kicad/amp/amp.kicad_sch (KiCad schematic)
At the start: 108 parts, among them J1 DC 12V IN, J2 IN L-G-R, J3 SPK L, J4 SPK R, Q1001 BC547, Q1002 BC547, Q1003 BC557, Q1004 BD139, Q1005 BD140, Q1006 BC547, Q2001 BC547, Q2002 BC547, Q2003 BC557, Q2004 BD139, Q2005 BD140, Q2006 BC547

Commit message: Release 1.2: mirror-loaded front end, closed-loop PSU, VU tap, headphone board
- Amp: PNP input pair with NPN current-mirror load, LED-referenced current-source tail,
  NPN VAS with bootstrapped load from +12V, 220p Miller + 47p lead cap (THD 0.004% at 26 mW/8R,
  0.019% at 0.29 W; was 0.03 / 0.2). 1k VU meter tap per channel to header J5.
- PSU: BC547 error amplifier, 5.6 V zener fed from VOUT, 8.2k + 2k trimmer / 10k divider,
  2.2k drive, 47n/100n compensation. 12.0 V set point, 0.14 V dip on a 1 A step.
- New headphone board (DPDT switch, 120R series, DIRECT jumpers, 3.5 mm jack, panel-jack header).
- Boards: amp 134x85 / compact 100x98, PSU 90x58, hp 42x30; panel 155x155 with four boards.
  All 2-layer boards and the panel DRC clean; single-sided amp down to 15 errors.
- Toolchain: STAMP constant, reroute.sh second routing pass, rotated titles, link holes on
  jumper pads, 2 mm routing corridor per channel.
- Docs, BOMs, order guide, changelog, known issues rewritten for release 2.
Parts:
- removed Q1001, Q1002, Q2001, Q2002: BC547, Custom:TO92_SOT23, symbol Transistor_BJT:BC547
- removed Q1003, Q2003: BC557, Custom:TO92_SOT23, symbol Transistor_BJT:BC557
- added C10008, C20008: 47p, Custom:C_P5_1206, symbol Device:C
- added D10001, D20001: LED red, LED_THT:LED_D3.0mm, symbol Device:LED
- added J5: VU L-G-R, Connector_PinHeader_2.54mm:PinHeader_1x03_P2.54mm_Vertical, symbol Connector_Generic:Conn_01x03
- added Q1001, Q1002, Q1009, Q2001, Q2002, Q2009: BC557, Custom:TO92_SOT23, symbol Transistor_BJT:BC557
- added Q1003, Q1007, Q1008, Q2003, Q2007, Q2008: BC547, Custom:TO92_SOT23, symbol Transistor_BJT:BC547
- added R10016, R10017, R20016, R20017: 100, Custom:R_Axial_1206, symbol Device:R
- added R10018, R20018: 1k, Custom:R_Axial_1206, symbol Device:R
- added TP1004, TP2004: LED 10.2V, TestPoint:TestPoint_Loop_D2.50mm_Drill1.0mm, symbol Connector:TestPoint
- C10004, C20004: value 100p -> 220p
- R10004, R20004: value 4.7k -> 1.2k
- R10005, R20005: value 10k -> 4.7k
- TP1001, TP2001: value B1 5.9V -> B1 6.1V
Connections:
- net +12V: now also R10011.1, R20011.1, D10001.2 (A), D20001.2 (A); no longer R10008.1, R20008.1
- net B5_L: now also C10004.1, Q1003.1 (C); no longer R10011.1
- net B5_R: now also C20004.1, Q2003.1 (C); no longer R20011.1
- net GND: now also R10008.2, R20008.2, J5.2 (Pin_2), R10016.2, R10017.2, R20016.2, R20017.2; no longer R10012.2, R20012.2
- net OUT_L: now also C10005.2, C10008.2; no longer C10005.1
- net OUT_R: now also C20005.2, C20008.2; no longer C20005.1
- net SPK_L: now also R10018.1
- net SPK_R: now also R20018.1
- net VAS_L: now also R10012.2; no longer C10004.1
- net VAS_R: now also R20012.2; no longer C20004.1
- net at C20004.2: now also Q2001.1 (C), Q2003.2 (B), Q2007.1 (C); no longer R20004.2
- net at C20001.1, R20003.2, TP2001.1: now also Q2001.2 (B)
- net at R20006.1, R20007.1: now also C20008.1, Q2002.2 (B)
- net at R20005.1: now also D20001.1 (K), Q2009.2 (B), TP2004.1
- net at R20011.2, R20012.1: now also C20005.1; no longer C20005.2
- net at R10004.2: now also Q1009.3 (E); no longer C10004.2
- net at C10001.1, R10003.2, TP1001.1: now also Q1001.2 (B)
- net at R10005.1: now also D10001.1 (K), Q1009.2 (B), TP1004.1
- net at R10006.1, R10007.1: now also C10008.1, Q1002.2 (B)
- net at R10011.2, R10012.1: now also C10005.1; no longer C10005.2
- new net: Q2002.1 (C), Q2007.2 (B), Q2008.1 (C), Q2008.2 (B)
- new net: Q2007.3 (E), R20016.1
- new net: Q1001.3 (E), Q1002.3 (E), Q1009.1 (C)
- new net: Q2003.3 (E), R20008.1
- new net: Q2001.3 (E), Q2002.3 (E), Q2009.1 (C)
- new net: Q1002.1 (C), Q1007.2 (B), Q1008.1 (C), Q1008.2 (B)
- new net: Q1008.3 (E), R10017.1
- new net: C10004.2, Q1001.1 (C), Q1003.2 (B), Q1007.1 (C)
- new net: Q1003.3 (E), R10008.1
- new net: Q1007.3 (E), R10016.1
- new net: Q2008.3 (E), R20017.1
- new net: Q2009.3 (E), R20004.2
- new net VU_L: J5.1 (Pin_1), R10018.2
- new net VU_R: J5.3 (Pin_3), R20018.2
Other:
- note added: "J5: VU meter tap, 1k in series with each speaker node (2.8 Vrms at 1 W / 8 ohm, no DC). Leave open if unused."
- note added: "Shared: DC in, reservoir, input header (L G R), speaker terminals, VU meter header (1k series from each speaker node). Test points TP1 +12V, TP2 GND."
- note removed: "Shared: DC in, reservoir, input header (L G R), speaker terminals. Test points TP1 +12V, TP2 GND."
- title: Stereo class-AB amplifier - BD139/BD140 outputs, 12 V -> Stereo class-AB amplifier (release 2) - mirror-loaded PNP input, NPN VAS, BD139/BD140 outputs, 12 V
