File: kicad/psu/psu.kicad_sch (KiCad schematic)
At the start: 30 parts, among them J1 AC IN 12-15V, J2 DC IN 12V, J3 DC OUT 1, J4 DC OUT 2, J5 LED REMOTE, Q1 BC547, Q2 TIP41C, Q3 BC547

Commit message: Release 1.2: mirror-loaded front end, closed-loop PSU, VU tap, headphone board
- Amp: PNP input pair with NPN current-mirror load, LED-referenced current-source tail,
  NPN VAS with bootstrapped load from +12V, 220p Miller + 47p lead cap (THD 0.004% at 26 mW/8R,
  0.019% at 0.29 W; was 0.03 / 0.2). 1k VU meter tap per channel to header J5.
- PSU: BC547 error amplifier, 5.6 V zener fed from VOUT, 8.2k + 2k trimmer / 10k divider,
  2.2k drive, 47n/100n compensation. 12.0 V set point, 0.14 V dip on a 1 A step.
- New headphone board (DPDT switch, 120R series, DIRECT jumpers, 3.5 mm jack, panel-jack header).
- Boards: amp 134x85 / compact 100x98, PSU 90x58, hp 42x30; panel 155x155 with four boards.
  All 2-layer boards and the panel DRC clean; single-sided amp down to 15 errors.
- Toolchain: STAMP constant, reroute.sh second routing pass, rotated titles, link holes on
  jumper pads, 2 mm routing corridor per channel.
- Docs, BOMs, order guide, changelog, known issues rewritten for release 2.
Parts:
- added C6: 47n, Custom:C_P5_1206, symbol Device:C
- added C7: 100n, Custom:C_P5_1206, symbol Device:C
- added Q4: BC547, Custom:TO92_SOT23, symbol Transistor_BJT:BC547
- added R5: 8.2k, Custom:R_Axial_1206, symbol Device:R
- added R6: 10k, Custom:R_Axial_1206, symbol Device:R
- added R7: 2.2k, Custom:R_Axial_1206, symbol Device:R
- added RV1: 2k, Potentiometer_THT:Potentiometer_Bourns_3296W_Vertical, symbol Device:R_Potentiometer_Trim
- added TP5: FB 6.3V, TestPoint:TestPoint_Loop_D2.50mm_Drill1.0mm, symbol Connector:TestPoint
- C3: value 100u -> 10u; footprint Capacitor_THT:CP_Radial_D6.3mm_P2.50mm -> Custom:CE_P2_1206
- D5: value 13V 1W -> 5.6V
- TP2: value VZ 13V -> VZ 5.6V
- TP3: value VOUT 11.5V -> VOUT 12.0V
Connections:
- net GND: now also R6.2
- net at C1.1, C2.1, D1.1 (K)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: now also R7.1; no longer R2.1
- net at C4.1, C5.1, D6.2 (A)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: now also R2.1, C7.1, R5.1
- net VZ: no longer names the net of C3.1, D5.1 (K), R2.2, TP2.1
- net VZ: now also Q4.3 (E); no longer Q1.2 (B), Q3.1 (C)
- new net: C6.2, C7.2, Q4.2 (B), R6.1, RV1.2, RV1.3, TP5.1
- new net: R5.2, RV1.1
- new net BQ1: C6.1, Q1.2 (B), Q3.1 (C), Q4.1 (C), R7.2
Other:
- note added: "Pass transistor Q2 needs a heatsink: 3.5 W at 15 VAC / 0.8 A, 3.9 W at 1.2 A (psu2.cir)."
- note added: "Regulator: Q4 compares FB (R5 + RV1 / R6 divider of VOUT) with the 5.6 V zener and pulls the driver base down through BQ1. RV1 sets VOUT, 11.4 to 12.7 V."
- note added: "Transformer secondary 12-15 VAC, 1.5 A or more for full stereo power (12 VAC: 12 V regulated up to 0.4 A, then follows the raw rail)."
- note removed: "Pass transistor Q2 needs a heatsink: 1.6 W at 12 VAC / 1 A, 4.9 W at 15 VAC / 1.1 A (psu.cir)."
- note removed: "Transformer secondary 12-15 VAC, 1.5 A or more for full stereo power (12 VAC: regulated to 0.35 A)."
- title: Discrete 12 V power supply - bridge, zener reference, TIP41C pass, DC-in bypass -> Discrete 12 V power supply (release 2) - bridge, closed-loop TIP41C regulator, DC-in bypass
