File: kicad/hp/hp.kicad_pcb (KiCad board)
At the start: 2 copper layers, 42 x 30 mm, 13 parts, among them J1 FROM AMP L-G-R, J2 SPK L, J3 SPK R, J4 3.5mm TRS, J5 PANEL JACK T-G-R, SW1 SPK / HP

Commit message: Headphone jack sleeve pad was left without its GND net
pcbgen stripped the SMD-twin suffix from every pad number ending in S, which turned the jack's
sleeve pad "S" into an empty key. Exact pad numbers are matched first now. Headphone boards,
panel, images and the release zip rebuilt; single-layer headphone board 3 wire links, clean.
Connections:
- J4 pad S: (no net) -> GND
Routing:
- net GND: track 41.4 -> 63.6 mm
