File: kicad/panel/stereo-panel.kicad_pcb (KiCad board)
At the start: 2 copper layers, 155.2 x 155.2 mm, 401 parts, among them J1 AC IN 12-15V, J1 DC 12V IN, J1 FROM AMP L-G-R, J1 IN L-G-R, J2 DC IN 12V, J2 IN L-G-R, J2 OUT L-G-R, J2 SPK L, J3 DC OUT 1, J3 LED IN, J3 SPK L, J3 SPK R, J4 3.5mm TRS, J4 DC OUT 2, J4 SPK R, J5 LED REMOTE, J5 PANEL JACK T-G-R, J5 VU L-G-R, Q1 BC547, Q1001 BC557, Q1002 BC557, Q1003 BC547, Q1004 BD139, Q1005 BD140, Q1006 BC547, Q1007 BC547, Q1008 BC547, Q1009 BC557, Q2 TIP41C, Q2001 BC557, Q2002 BC557, Q2003 BC547, Q2004 BD139, Q2005 BD140, Q2006 BC547, Q2007 BC547, Q2008 BC547, Q2009 BC557, Q3 BC547, Q4 BC547, SW1 SPK / HP

Commit message: Headphone jack sleeve pad was left without its GND net
pcbgen stripped the SMD-twin suffix from every pad number ending in S, which turned the jack's
sleeve pad "S" into an empty key. Exact pad numbers are matched first now. Headphone boards,
panel, images and the release zip rebuilt; single-layer headphone board 3 wire links, clean.
Connections:
- J4 pad S: (no net) -> Board_2-GND
Routing:
- net Board_2-GND: track 41.4 -> 63.6 mm
